File: OBS-buttons-buttons.brd (EAGLE design)
At the start: 144.8 x 81.2 mm, 23 parts

Commit message: initial prototype
Parts:
- removed BOARD1, BOARD2: (no value), SPCoast:BOARD-SEEED10X5-NOHOLES
- removed J3, J4: (no value), SPCoast:1X08_LOCK
- removed R1, R2, R3, R4, R5, R6: (no value), SPCoast:AXIAL-0.4-RES
- removed U$1: ARDUINO-PRO-MICROEBAY, SPCoast:ARDUINO-PRO-MICRO
- moved J2 100.3 mm to (34.3, 6.35)
- moved J1 100.3 mm to (15.2, 57.1)
- moved LED1 100.3 mm to (40.6, 48.3)
- moved LED2 100.3 mm to (8.89, 48.3)
- moved LED3 100.3 mm to (40.6, 35.6)
- moved LED4 100.3 mm to (8.89, 35.6)
- moved LED5 100.3 mm to (40.6, 24.1)
- moved LED6 100.3 mm to (8.89, 24.1)
- moved SW1 100.3 mm to (24.0, 48.0)
- moved SW2 100.3 mm to (24.0, 36.0)
- moved SW3 100.3 mm to (24.0, 24.0)
- moved CON1 100.3 mm to (39.4, 59.7)
Connections:
- removed net I1: J3.5, U$1.AD0
- removed net I2: J3.4, U$1.D13
- removed net I3: J3.3, U$1.D12
- removed net I4: J3.2, U$1.D11
- removed net I5: J3.6, U$1.D8
- removed net I6: J3.7, U$1.D4
- removed net I7: J3.8, U$1.D2
- removed net N$1: LED1.K, R1.P$2
- removed net N$2: LED2.K, R2.P$2
- removed net N$3: LED3.K, R3.P$2
- removed net N$4: LED4.K, R4.P$2
- removed net N$5: LED5.K, R5.P$2
- removed net N$6: LED6.K, R6.P$2
- removed net O1: J4.1, U$1.D3
- removed net O2: J4.2, U$1.D5
- removed net O3: J4.3, U$1.D6
- removed net O4: J4.4, U$1.D7
- removed net O5: J4.5, U$1.D9
- removed net O6: J4.6, U$1.D10
- net CUT-LED: now also LED1.K; no longer R1.P$1
- net FADE-LED: now also LED2.K; no longer R2.P$1
- net GND: no longer J4.7, J4.8, U$1.GND@1, U$1.GND@2, U$1.GND@4
- net SCENE1-LED: now also LED3.K; no longer R3.P$1
- net SCENE2-LED: now also LED4.K; no longer R4.P$1
- net SCENE3-LED: now also LED5.K; no longer R5.P$1
- net SCENE4-LED: now also LED6.K; no longer R6.P$1
- net VCC: no longer J3.1, U$1.5V
Routing:
- net FADE-LED: track 9.72 -> 53.3 mm
- net O5: track 40.6 -> 0.00 mm
- net CUT-LED: track 8.27 -> 48.9 mm
- net O3: track 39.6 -> 0.00 mm
- net O2: track 39.3 -> 0.00 mm
- net O4: track 39.3 -> 0.00 mm
- net O1: track 38.5 -> 0.00 mm
- net N$1: track 36.9 -> 0.00 mm
- net N$2: track 35.9 -> 0.00 mm
- net I3: track 30.4 -> 0.00 mm
- net I1: track 30.4 -> 0.00 mm
- net I4: track 30.1 -> 0.00 mm
- net I2: track 30.1 -> 0.00 mm
- net SCENE2-LED: track 12.4 -> 40.7 mm
- net SCENE1-LED: track 10.6 -> 35.9 mm
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Other:
- board size 144.8 x 81.2 mm -> 44.5 x 62.2 mm
- board text removed: "2 Scene"
- board text removed: "4 Scene"
- board text removed: "Cut"
- board text removed: "Fade"
- board text removed: "Scene"
- board text removed: "Scene 1"
- board text removed: "Scene 3"
- board text removed: "Transition"
